Commit message: Update the correct urdf model

File: warrior_description/urdf/robot.urdf (robot description, URDF)
Before this commit: robot test_robot, 6 links, 5 joints
Links:
- removed link wheel_link
- removed link wheel_link2
- removed link wheel_link3
- added link front_drive_wheel_link, mass 0.5; collision mesh filename=file://$(find warrior_description)/meshes/drive_wheel.stl; visual mesh filename=file://$(find warrior_description)/meshes/drive_wheel.stl
- added link front_steer_wheel_link, mass 0.5; collision mesh filename=file://$(find warrior_description)/meshes/steer_wheel.stl; visual mesh filename=file://$(find warrior_description)/meshes/steer_wheel.stl
- added link left_drive_wheel_link, mass 0.5; collision mesh filename=file://$(find warrior_description)/meshes/drive_wheel.stl; visual mesh filename=file://$(find warrior_description)/meshes/drive_wheel.stl
- added link left_steer_wheel_link, mass 0.5; collision mesh filename=file://$(find warrior_description)/meshes/steer_wheel.stl; visual mesh filename=file://$(find warrior_description)/meshes/steer_wheel.stl
- added link right_drive_wheel_link, mass 0.5; collision mesh filename=file://$(find warrior_description)/meshes/drive_wheel.stl; visual mesh filename=file://$(find warrior_description)/meshes/drive_wheel.stl
- added link right_steer_wheel_link, mass 0.5; collision mesh filename=file://$(find warrior_description)/meshes/steer_wheel.stl; visual mesh filename=file://$(find warrior_description)/meshes/steer_wheel.stl
- link base_link: mass 15.0 -> 75.0; geometry collision mesh filename=file://$(find warrior_description)/meshes/warrior_base_with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; visual mesh filename=file://$(find warrior_description)/meshes/warrior_base_with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
Joints:
- removed joint base_to_wheel
- removed joint base_to_wheel2
- removed joint base_to_wheel3
- added joint front_drive_wheel_joint: type continuous, parent front_steer_wheel_link, child front_drive_wheel_link, origin xyz=0 0 -0.15 rpy=0 0 0, axis 1 0 0
- added joint front_steer_joint: type continuous, parent base_link, child front_steer_wheel_link, origin xyz=0.845 0 0 rpy=0 0 0, axis 0 0 1
- added joint left_drive_wheel_joint: type continuous, parent left_steer_wheel_link, child left_drive_wheel_link, origin xyz=0 0 -0.15 rpy=0 0 0, axis 1 0 0
- added joint left_steer_joint: type continuous, parent base_link, child left_steer_wheel_link, origin xyz=0 0.465 0 rpy=0 0 0, axis 0 0 1
- added joint right_drive_joint: type continuous, parent right_steer_wheel_link, child right_drive_wheel_link, origin xyz=0 0 -0.15 rpy=0 0 0, axis 1 0 0
- added joint right_steer_joint: type continuous, parent base_link, child right_steer_wheel_link, origin xyz=0 -0.465 0 rpy=0 0 0, axis 0 0 1

Commit message: The correct urdf draft

File: warrior_description/urdf/robot.urdf (robot description, URDF)
Before this commit: robot wsu_warrior, 9 links, 8 joints
Links:
- removed link pole_for_lidar
- added link pole_link
- link lidar_link: mass 1.0 -> None; geometry 
Joints:
- removed joint base_to_lidar_pole
- removed joint lidar_to_pole
- added joint base_to_pole: type fixed, parent base_link, child pole_link, origin xyz=0 0 0.9 rpy=0 0 0
- added joint lidar_joint: type fixed, parent pole_link, child lidar_link, origin xyz=0.36 0 0 rpy=0 0 0
- joint front_steer_joint: origin xyz=0.845 0 0 rpy=0 0 0 -> xyz=0.845 0 0 rpy=0 0 -1.5708
- joint left_steer_joint: origin xyz=0 0.465 0 rpy=0 0 0 -> xyz=0 0.465 0 rpy=0 0 -1.0472
- joint right_steer_joint: origin xyz=0 -0.465 0 rpy=0 0 0 -> xyz=0 -0.465 0 rpy=0 0 -2.0944
