Commit message: Fix some stuff

File: warrior_description/urdf/warrior.urdf.xacro (robot description, xacro)
@@ -1,5 +1,5 @@
 <?xml version="1.0"?>
 <robot xmlns:xacro="http://www.ros.org/wiki/xacro" name="wsu_warrior">
-    <xacro:include filename="$(find warrior_description)/xacro/warrior.ros2_control.xacro"/>
-    <xacro:include filename="$(find warrior_description)/xacro/warrior.xacro"/>
+    <xacro:include filename="$(find warrior_description)/xacro/robot.ros2_control.xacro"/>
+    <xacro:include filename="$(find warrior_description)/xacro/robot.xacro"/>
 </robot>

File: warrior_description/xacro/gzsim.ros2_control.xacro (robot description, xacro)
@@ -1,44 +1,4 @@
 <?xml version="1.0"?>
 <robot xmlns:xacro="http://www.ros.org/wiki/xacro">
-    <!-- Gazebo colors -->
-    <gazebo reference="base_link">
-        <material>Gazebo/Grey</material>
-    </gazebo>
-    <gazebo reference="left_steer_wheel_link">
-        <material>Gazebo/Blue</material>
-    </gazebo>
-    <gazebo reference="right_steer_wheel_link">
-        <material>Gazebo/Green</material>
-    </gazebo>
-    <gazebo reference="front_steer_wheel_link">
-        <material>Gazebo/Cyan</material>
-    </gazebo>
-    <gazebo reference="left_drive_wheel_link">
-        <material>Gazebo/DarkGrey</material>
-        <mu1>0.8</mu1>
-        <mu2>0.8</mu2>
-        <kp>1000000.0</kp>
-        <kd>100.0</kd>
-        <minDepth>0.001</minDepth>
-        <maxVel>1.0</maxVel>
-    </gazebo>
-    <gazebo reference="right_drive_wheel_link">
-        <material>Gazebo/DarkGrey</material>
-        <mu1>0.8</mu1>
-        <mu2>0.8</mu2>
-        <kp>1000000.0</kp>
-        <kd>100.0</kd>
-        <minDepth>0.001</minDepth>
-        <maxVel>1.0</maxVel>
-    </gazebo>
-    <gazebo reference="front_drive_wheel_link">
-        <material>Gazebo/DarkGrey</material>
-        <mu1>0.8</mu1>
-        <mu2>0.8</mu2>
-        <kp>1000000.0</kp>
-        <kd>100.0</kd>
-        <minDepth>0.001</minDepth>
-        <maxVel>1.0</maxVel>
-    </gazebo>
     <!-- ros2_control configuration for diff drive -->
     <ros2_control name="warrior_gazebo_ros2_control" type="system">

File: warrior_description/xacro/robot.ros2_control.xacro (robot description, xacro)
@@ -1,5 +1,5 @@
 <?xml version="1.0"?>
-<robot xmlns:xacro="http://www.ros.org/wiki/xacro" name="wsu_warrior_ros2_control">
-    <ros2_control name="warrior_ros2_control" type="system">
+<robot xmlns:xacro="http://www.ros.org/wiki/xacro" name="robot_ros2_control">
+    <ros2_control name="robot_ros2_control" type="system">
         <hardware>
             <plugin>mock_components/GenericSystem</plugin>

File: warrior_description/xacro/robot.xacro (robot description, xacro)
@@ -208,28 +208,23 @@
   </joint>
   <!-- ========== Gazebo LiDAR Sensor ========== -->
-  <!-- <gazebo reference="lidar_link">
-    <sensor type="ray" name="lidar_sensor">
-      <pose>0 0 0 0 0 0</pose>
-      <update_rate>5.0</update_rate>
-      <ray>
-        <scan>
-          <horizontal>
-            <samples>180</samples>
-            <resolution>1</resolution>
-            <min_angle>-3.14</min_angle>
-            <max_angle>3.14</max_angle>
-          </horizontal>
-        </scan>
+  <gazebo reference="lidar_link">
+    <sensor name="lidar_sensor" type="gpu_lidar">
+      <update_rate>10.0</update_rate>
+      <lidar>
+        <horizontal>
+          <samples>720</samples>
+          <resolution>1</resolution>
+          <min_angle>-3.1415</min_angle>
+          <max_angle>3.1415</max_angle>
+        </horizontal>
         <range>
           <min>0.12</min>
-          <max>5</max>
-          <resolution>0.02</resolution>
+          <max>10.0</max>
+          <resolution>0.01</resolution>
         </range>
-      </ray>
-      <plugin name="gazebo_ros_laser_controller" filename="libgazebo_ros_laser.so">
-        <topicName>/scan</topicName>
-        <frameName>lidar_link</frameName>
-      </plugin>
+      </lidar>
+      <topic>/lidar</topic>
+      <visualize>true</visualize>
     </sensor>
-  </gazebo> -->
+  </gazebo>
 </robot>
