Commit message: Update code for new urdf

File: warrior_description/urdf/gzsim.urdf.xacro (robot description, xacro)
@@ -2,5 +2,5 @@
 <robot xmlns:xacro="http://www.ros.org/wiki/xacro" name="wsu_warrior_sim">
     <xacro:include filename="$(find warrior_description)/xacro/gazebo.xacro"/>
-    <xacro:include filename="$(find warrior_description)/xacro/gzsim.ros2_control.xacro"/>
+    <xacro:include filename="$(find warrior_description)/xacro/ros2_control/gzsim.ros2_control.xacro"/>
     <xacro:include filename="$(find warrior_description)/xacro/robot.xacro"/>
 </robot>

File: warrior_description/urdf/warrior.urdf.xacro (robot description, xacro)
@@ -1,5 +1,5 @@
 <?xml version="1.0"?>
 <robot xmlns:xacro="http://www.ros.org/wiki/xacro" name="wsu_warrior">
-    <xacro:include filename="$(find warrior_description)/xacro/robot.ros2_control.xacro"/>
+    <xacro:include filename="$(find warrior_description)/xacro/ros2_control/robot.ros2_control.xacro"/>
     <xacro:include filename="$(find warrior_description)/xacro/robot.xacro"/>
 </robot>

File: warrior_description/xacro/gazebo.xacro (robot description, xacro)
@@ -5,11 +5,11 @@
         <material>Gazebo/Grey</material>
     </gazebo>
-    <gazebo reference="left_steer_wheel_link">
+    <gazebo reference="left_steer_assembly_link">
         <material>Gazebo/Blue</material>
     </gazebo>
-    <gazebo reference="right_steer_wheel_link">
+    <gazebo reference="right_steer_assembly_link">
         <material>Gazebo/Green</material>
     </gazebo>
-    <gazebo reference="front_steer_wheel_link">
+    <gazebo reference="front_steer_assembly_link">
         <material>Gazebo/Cyan</material>
     </gazebo>

File: warrior_description/xacro/material.xacro (robot description, xacro)
@@ -1,16 +1,23 @@
 <?xml version="1.0"?>
 <robot xmlns:xacro="http://www.ros.org/wiki/xacro">
-   <xacro:property name="front_plate_offset" value="0.838 0.003 -0.349"/>
-   <xacro:property name="left_plate_offset" value="0.025 0.47 -0.349"/>
-   <xacro:property name="right_plate_offset" value="0.024 -0.468 -0.349"/>
-  <!-- ========== Material Definitions ========== -->
+  <!-- ========== Basic Colors ========== -->
   <material name="gray">
     <color rgba="0.5 0.5 0.5 1"/>
   </material>
+  <material name="dark_gray">
+    <color rgba="0.2 0.2 0.2 1"/>
+  </material>
+  <material name="light_gray">
+    <color rgba="0.8 0.8 0.8 1"/>
+  </material>
+  <material name="white">
+    <color rgba="1.0 1.0 1.0 1"/>
+  </material>
+  <material name="black">
+    <color rgba="0.0 0.0 0.0 1"/>
+  </material>
+  <!-- ========== Saturated Colors ========== -->
   <material name="blue">
     <color rgba="0.0 0.0 1.0 1"/>
-  </material>
-  <material name="yellow">
-    <color rgba="1.0 1.0 0.0 1"/>
   </material>
   <material name="green">
@@ -20,4 +27,7 @@
     <color rgba="1.0 0.0 0.0 1"/>
   </material>
+  <material name="yellow">
+    <color rgba="1.0 1.0 0.0 1"/>
+  </material>
   <material name="cyan">
     <color rgba="0.0 1.0 1.0 1"/>
@@ -26,3 +36,35 @@
     <color rgba="1.0 0.0 1.0 1"/>
   </material>
+  <material name="orange">
+    <color rgba="1.0 0.5 0.0 1"/>
+  </material>
+  <material name="purple">
+    <color rgba="0.5 0.0 0.8 1"/>
+  </material>
+  <!-- ========== Low-Saturation Engineering Colors ========== -->
+  <material name="steel_blue">
+    <color rgba="0.27 0.51 0.71 1"/>
+  </material>
+  <material name="olive">
+    <color rgba="0.5 0.5 0.0 1"/>
+  </material>
+  <material name="teal">
+    <color rgba="0.0 0.5 0.5 1"/>
+  </material>
+  <material name="brown">
+    <color rgba="0.4 0.26 0.13 1"/>
+  </material>
+  <material name="pink">
+    <color rgba="1.0 0.75 0.8 1"/>
+  </material>
+  <!-- ========== Metallic / Robotics Colors ========== -->
+  <material name="silver">
+    <color rgba="0.75 0.75 0.75 1"/>
+  </material>
+  <material name="gold">
+    <color rgba="1.0 0.84 0.0 1"/>
+  </material>
+  <material name="copper">
+    <color rgba="0.72 0.45 0.20 1"/>
+  </material>
 </robot>

File: warrior_description/xacro/swerve_module/constant.xacro (robot description, xacro)
@@ -1,13 +1,12 @@
 <?xml version="1.0"?>
 <robot xmlns:xacro="http://www.ros.org/wiki/xacro">
-  <!-- <xacro:include filename="$(find warrior_description)/xacro/material.xacro"/> -->
+   <!-- <xacro:include filename="$(find warrior_description)/xacro/material.xacro"/> -->
    <xacro:property name="slewing_plate_mass" value="0.5"/>
    <xacro:property name="steer_assembly_mass" value="0.7"/>
-   <xacro:property name="steer_assembly_color" value="gray"/>
-   <xacro:property name="slewing_plate_color" value="gray"/>
+   <xacro:property name="steer_assembly_color" value="light_gray"/>
+   <xacro:property name="slewing_plate_color" value="silver"/>
+   <xacro:property name="drive_wheel_color" value="cyan"/>
    <xacro:property name="swerve_offset_to_plate" value="0 0 -0.011"/>
    <xacro:property name="drive_wheel_offset" value="0.025 0 -0.147"/>
-    <xacro:property name="steer_color" value="cyan"/>
-    <xacro:property name="drive_color" value="gray"/>
     <xacro:property name="drive_rpy" value="0 0 0"/>
     <xacro:property name="drive_axis" value="1 0 0"/>

File: warrior_description/xacro/swerve_module/swerve_module.xacro (robot description, xacro)
@@ -57,5 +57,5 @@
           <mesh filename="file://$(find warrior_description)/meshes/drive_wheel.stl"/>
         </geometry>
-        <material name="${drive_color}"/>
+        <material name="${drive_wheel_color}"/>
       </visual>
       <collision>

Commit message: Add lidar scan in Gazebo

File: warrior_description/urdf/gzsim.urdf.xacro (robot description, xacro)
@@ -1,5 +1,5 @@
 <?xml version="1.0"?>
 <robot xmlns:xacro="http://www.ros.org/wiki/xacro" name="wsu_warrior_sim">
-    <xacro:include filename="$(find warrior_description)/xacro/gazebo.xacro"/>
+    <xacro:include filename="$(find warrior_description)/xacro/material.gazebo.xacro"/>
     <xacro:include filename="$(find warrior_description)/xacro/ros2_control/gzsim.ros2_control.xacro"/>
     <xacro:include filename="$(find warrior_description)/xacro/robot.xacro"/>

File: warrior_description/xacro/robot.xacro (robot description, xacro)
@@ -1,6 +1,8 @@
 <?xml version="1.0"?>
 <robot name="warrior_robot" xmlns:xacro="http://www.ros.org/wiki/xacro">
+  <!-- ========== Includes ========== -->
   <xacro:include filename="$(find warrior_description)/xacro/material.xacro"/>
   <xacro:include filename="$(find warrior_description)/xacro/swerve_module/swerve_module.xacro"/>
+  <xacro:include filename="$(find warrior_description)/xacro/sensors/lidar.xacro"/>
   <!-- ========== Properties ========== -->
   <xacro:property name="angle_offset" value="${pi/6}"/>
@@ -90,32 +92,7 @@
     <origin xyz="0 0 ${pole_height}" rpy="${pi} 0 0"/>
   </joint>
-  <!-- ========== LiDAR Link ========== -->
-  <link name="lidar_link">
-    <visual>
-      <origin xyz="0 -0.015 0" rpy="0 0 0"/>
-      <geometry>
-        <mesh filename="file://$(find warrior_description)/meshes/unitree_lidar.stl"/>
-      </geometry>
-      <material name="black">
-          <color rgba="0 0 0 1"/>
-      </material>
-    </visual>
-    <collision>
-      <origin xyz="0 -0.015 0" rpy="0 0 0"/>
-      <geometry>
-        <mesh filename="file://$(find warrior_description)/meshes/unitree_lidar.stl"/>
-      </geometry>
-    </collision>
-    <inertial>
-      <origin xyz="0 -0.015 0" rpy="0 0 0"/>
-      <mass value="1.0"/>
-      <inertia ixx="0.01" ixy="0" ixz="0" iyy="0.01" iyz="0" izz="0.005"/>
-    </inertial>
-  </link>
-  <joint name="lidar_joint" type="fixed">
-    <parent link="pole_link"/>
-    <child link="lidar_link"/>
-    <origin xyz="0.32 0 0.05" rpy="0 0 0"/>
-  </joint>
+  <!-- ========== LiDAR Sensor ========== -->
+  <xacro:lidar_macro parent="pole_link" lidar_name="L1_lidar"
+                     xyz="${lidar_offset_x} 0 0" rpy="0 0 0" mass="0.5"/>
   <!-- ========== Camera Link ========= -->
   <link name="camera_link">
@@ -146,24 +123,3 @@
     <origin xyz="0.32 0 0" rpy="0 0 0"/>
   </joint>
-  <!-- ========== Gazebo LiDAR Sensor ========== -->
-  <gazebo reference="lidar_link">
-    <sensor name="lidar_sensor" type="gpu_lidar">
-      <update_rate>10.0</update_rate>
-      <lidar>
-        <horizontal>
-          <samples>720</samples>
-          <resolution>1</resolution>
-          <min_angle>-3.1415</min_angle>
-          <max_angle>3.1415</max_angle>
-        </horizontal>
-        <range>
-          <min>0.12</min>
-          <max>10.0</max>
-          <resolution>0.01</resolution>
-        </range>
-      </lidar>
-      <topic>/lidar</topic>
-      <visualize>true</visualize>
-    </sensor>
-  </gazebo>
 </robot>

File: warrior_description/xacro/sensors/lidar.xacro (robot description, xacro)
@@ -1,46 +1,72 @@
 <?xml version="1.0"?>
-<robot xmlns:xacro="http://www.ros.org/wiki/xacro" >
-  <joint name="laser_joint" type="fixed">
-    <parent link="base_link"/>
-    <child link ="laser_frame"/>
-    <origin xyz="0 0 ${base_height + lidar_length}"/>
-  </joint>
-  <link name="laser_frame">
-    <visual name="laser_visual">
-      <geometry>
-          <cylinder length="${lidar_length}" radius="${lidar_radius}" />
-      </geometry>
-      <material name="blue"/>
-    </visual>
-    <collision name="laser_collision">
-      <geometry>
-          <cylinder length="${lidar_length}" radius="${lidar_radius}" />
-      </geometry>
-    </collision>
-    <xacro:inertial_cylinder mass="0.1" length="0.05" radius="0.05">
-        <origin xyz="0 0 0" rpy="0 0 0"/>
-    </xacro:inertial_cylinder>
-  </link>
-<gazebo reference="laser_frame">
-  <sensor name="laser" type="gpu_lidar">
-    <pose>0 0 0 0 0 0</pose>
-    <update_rate>10</update_rate>
-    <visualize>true</visualize>
-    <lidar>
-      <scan>
-        <horizontal>
-          <samples>360</samples>
-          <min_angle>-3.14</min_angle>
-          <max_angle>3.14</max_angle>
-        </horizontal>
-      </scan>
-      <range>
-        <min>0.3</min>
-        <max>12.0</max>
-      </range>
-    </lidar>
-    <topic>scan</topic>
-    <gz_frame_id>laser_frame</gz_frame_id>
-  </sensor>
-</gazebo>
+<robot xmlns:xacro="http://www.ros.org/wiki/xacro">
+  <!-- ========== LiDAR Macro ========== -->
+  <xacro:macro name="lidar_macro" params="parent lidar_name xyz rpy:='0 0 0' mass:=1.0">
+    <!-- LiDAR Link -->
+    <link name="${lidar_name}_link">
+      <visual>
+        <origin xyz="0 -0.015 0" rpy="0 0 0"/>
+        <geometry>
+          <mesh filename="file://$(find warrior_description)/meshes/unitree_lidar.stl"/>
+        </geometry>
+        <material name="black"/>
+      </visual>
+      <collision>
+        <origin xyz="0 -0.015 0" rpy="0 0 0"/>
+        <geometry>
+          <mesh filename="file://$(find warrior_description)/meshes/unitree_lidar.stl"/>
+        </geometry>
+      </collision>
+      <inertial>
+        <origin xyz="0 -0.015 0" rpy="0 0 0"/>
+        <mass value="${mass}"/>
+        <inertia ixx="0.01" ixy="0" ixz="0" iyy="0.01" iyz="0" izz="0.005"/>
+      </inertial>
+    </link>
+    <!-- LiDAR Joint -->
+    <joint name="${lidar_name}_joint" type="fixed">
+      <parent link="${parent}"/>
+      <child link="${lidar_name}_link"/>
+      <origin xyz="${xyz}" rpy="${rpy}"/>
+    </joint>
+    <!-- Gazebo Sensor Plugin -->
+    <gazebo reference="${lidar_name}_link">
+      <plugin filename="gz-sim-sensors-system" name="gz::sim::systems::Sensors">
+        <render_engine>ogre</render_engine>
+      </plugin>
+      <sensor name="${lidar_name}" type="gpu_lidar">
+        <topic>${lidar_name}/scan</topic>
+        <update_rate>10</update_rate>
+        <gz_frame_id>${lidar_name}_link</gz_frame_id>
+        <ray>
+          <scan>
+            <horizontal>
+              <samples>720</samples>
+              <resolution>1</resolution>
+              <min_angle>-3.14</min_angle>
+              <max_angle>3.14</max_angle>
+            </horizontal>
+            <vertical>
+              <samples>16</samples>
+              <resolution>1</resolution>
+              <min_angle>0</min_angle>
+              <max_angle>1.041799</max_angle>
+            </vertical>
+          </scan>
+          <range>
+            <min>0.05</min>
+            <max>2.5</max>
+            <resolution>0.01</resolution>
+          </range>
+        </ray>
+        <noise>
+          <type>gaussian</type>
+          <mean>0.0</mean>
+          <stddev>0.01</stddev>
+        </noise>
+        <always_on>1</always_on>
+        <visualize>true</visualize>
+      </sensor>
+    </gazebo>
+  </xacro:macro>
 </robot>
