Commit message: Update swerve module

File: warrior_description/xacro/material.gazebo.xacro (robot description, xacro)
@@ -41,3 +41,10 @@
         <maxVel>1.0</maxVel>
     </gazebo>
+    <gazebo reference="beacon_light_link">
+        <material>Gazebo/Red</material>
+        <ambient>1.0 0.5 0.0 1</ambient>
+        <diffuse>1.0 0.5 0.0 1</diffuse>
+        <specular>1.0 0.6 0.1 1</specular>
+        <emissive>1.5 0.5 0.0 1</emissive>
+    </gazebo>
 </robot>

File: warrior_description/xacro/material.xacro (robot description, xacro)
@@ -42,4 +42,7 @@
     <color rgba="1.0 0.5 0.0 1"/>
   </material>
+  <material name="warning_orange">
+    <color rgba="0.9 0.35 0.05 0.75"/>
+  </material>
   <material name="purple">
     <color rgba="0.5 0.0 0.8 1"/>

File: warrior_description/xacro/robot.xacro (robot description, xacro)
@@ -28,8 +28,7 @@
   <!-- lidar properties -->
   <xacro:property name="pole_height" value="0.527"/>
-  <xacro:property name="lidar_offset_x" value="0.32"/>
-  <xacro:property name="lidar_offset_z" value="0.005"/>
+  <xacro:property name="lidar_offset" value="0.135 -0.005 0.075"/>
   <!-- camera properties -->
-  <xacro:property name="camera_offset" value="0.32 0.0 -0.115"/>
+  <xacro:property name="camera_offset" value="0.415 0.0 -0.015"/>
   <!-- ========== Base Footprint Link ========== -->
   <link name="base_footprint"/>
@@ -94,7 +93,33 @@
   <!-- ========== LiDAR Sensor ========== -->
   <xacro:lidar_macro parent="pole_link" lidar_name="L1_lidar"
-                     xyz="${lidar_offset_x} 0 ${lidar_offset_z}" rpy="0 0 3.1415" mass="0.5"/>
+                     xyz="${lidar_offset}" rpy="0 0 3.1415" mass="0.5"/>
   <!-- ========== Camera Sensor ========== -->
   <xacro:camera_macro parent="pole_link" camera_name="insta360_camera"
                       xyz="${camera_offset}" rpy="${pi} 0 0" mass="0.5"/>
+  <!-- ========== Beacon Light ========== -->
+  <link name="beacon_light_link">
+    <visual>
+      <origin xyz="0 0 0" rpy="3.1415 0 0"/>
+      <geometry>
+        <mesh filename="file://$(find warrior_description)/meshes/beacon_light.stl"/>
+      </geometry>
+      <material name="warning_orange"/>
+    </visual>
+    <collision>
+      <origin xyz="0 0 0" rpy="3.1415 0 0"/>
+      <geometry>
+        <mesh filename="file://$(find warrior_description)/meshes/beacon_light.stl"/>
+      </geometry>
+    </collision>
+    <inertial>
+      <origin xyz="0 0 0" rpy="0 0 0"/>
+      <mass value="0.5"/>
+      <inertia ixx="0.01" ixy="0" ixz="0" iyy="0.01" iyz="0" izz="0.01"/>
+    </inertial>
+  </link>
+  <joint name="base_to_beacon_light" type="fixed">
+    <parent link="pole_link"/>
+    <child link="beacon_light_link"/>
+    <origin xyz="0.135 0.0 -0.022" rpy="0 0 0"/>
+  </joint>
 </robot>

File: warrior_description/xacro/sensors/camera.xacro (robot description, xacro)
@@ -5,5 +5,5 @@
   <link name="camera_link">
     <visual>
-      <origin xyz="0 0 0" rpy="${pi/2} 0 -${pi/2}"/>
+      <origin xyz="0 0 0" rpy="0 0 -${pi/2}"/>
       <geometry>
         <mesh filename="file://$(find warrior_description)/meshes/insta360_camera.stl"/>
@@ -14,5 +14,5 @@
     </visual>
     <collision>
-      <origin xyz="0 0 0" rpy="${pi/2} 0 -${pi/2}"/>
+      <origin xyz="0 0 0" rpy="0 0 -${pi/2}"/>
       <geometry>
         <mesh filename="file://$(find warrior_description)/meshes/insta360_camera.stl"/>

File: warrior_description/xacro/sensors/imu.xacro (robot description, xacro)
@@ -15,5 +15,5 @@
         <box size="${imu_length} ${imu_width} ${imu_height}" />
       </geometry>
-      <material name="orange"/>
+      <material name="cyan"/>
     </visual>
   </link>
