Commit message: Update simulation pipeline

File: warrior_description/xacro/material.xacro (robot description, xacro)
@@ -7,4 +7,7 @@
   <material name="dark_gray">
     <color rgba="0.2 0.2 0.2 1"/>
+  </material>
+  <material name="medium_gray">
+    <color rgba="0.55 0.55 0.55 1"/>
   </material>
   <material name="light_gray">

File: warrior_description/xacro/robot.xacro (robot description, xacro)
@@ -6,4 +6,6 @@
   <xacro:include filename="$(find warrior_description)/xacro/sensors/lidar.xacro"/>
   <xacro:include filename="$(find warrior_description)/xacro/sensors/camera.xacro"/>
+  <xacro:include filename="$(find warrior_description)/xacro/sensors/imu.xacro"/>
+  <!-- <xacro:include filename="$(find warrior_description)/xacro/sensors/gps.xacro"/> -->
   <!-- ========== Properties ========== -->
   <xacro:property name="angle_offset" value="${pi/6}"/>
@@ -12,9 +14,11 @@
    <xacro:property name="right_plate_offset" value="0.024 -0.468 -0.349"/>
   <!-- Wheel properties -->
-  <xacro:property name="wheel_mass" value="0.5"/>
+  <!-- <xacro:property name="wheel_mass" value="2.5"/> -->
+  <xacro:property name="wheel_mass" value="5.0"/>
   <xacro:property name="wheel_offset_z" value="-0.15"/>
   <xacro:property name="wheel_radius" value="0.1"/>
   <!-- Base properties -->
-  <xacro:property name="base_mass" value="0.5"/>
+  <!-- <xacro:property name="base_mass" value="6.0"/> -->
+  <xacro:property name="base_mass" value="10.0"/>
   <xacro:property name="base_footprint_height" value="${0.508 + wheel_radius}"/>
   <!-- Initial orientations (radians) -->
@@ -42,5 +46,5 @@
         <mesh filename="file://$(find warrior_description)/meshes/warrior_body.stl"/>
       </geometry>
-      <material name="gray"/>
+      <material name="medium_gray"/>
     </visual>
     <collision>
@@ -90,5 +94,5 @@
   <!-- ========== LiDAR Sensor ========== -->
   <xacro:lidar_macro parent="pole_link" lidar_name="L1_lidar"
-                     xyz="${lidar_offset_x} 0 ${lidar_offset_z}" rpy="0 0 0" mass="0.5"/>
+                     xyz="${lidar_offset_x} 0 ${lidar_offset_z}" rpy="0 0 3.1415" mass="0.5"/>
   <!-- ========== Camera Sensor ========== -->
   <xacro:camera_macro parent="pole_link" camera_name="insta360_camera"

File: warrior_description/xacro/ros2_control/gzsim.ros2_control.xacro (robot description, xacro)
@@ -47,4 +47,17 @@
             <parameters>$(find warrior_control)/config/warrior_controllers.yaml</parameters>
         </plugin>
+        <plugin filename="gz-sim-imu-system" name="gz::sim::systems::Imu"/>
+        <!-- <plugin filename="gz-sim-forcetorque-system" name="gz::sim::systems::ForceTorque"/> -->
+        <plugin filename="ignition-gazebo-forcetorque-system" name="ignition::gazebo::systems::ForceTorque"/>
+        <plugin filename="gz-sim-contact-system" name="gz::sim::systems::Contact"/>
+        <plugin filename="gz-sim-touchplugin-system" name="gz::sim::systems::TouchPlugin">
+        <target>vehicle_blue</target>
+        <namespace>wall</namespace>
+        <time>0.001</time>
+        <enabled>true</enabled>
+        </plugin>
+        <plugin filename="gz-sim-sensors-system" name="gz::sim::systems::Sensors">
+        <render_engine>ogre</render_engine>
+        </plugin>
     </gazebo>
 </robot>

File: warrior_description/xacro/sensors/camera.xacro (robot description, xacro)
@@ -9,6 +9,6 @@
         <mesh filename="file://$(find warrior_description)/meshes/insta360_camera.stl"/>
       </geometry>
-      <material name="light_grey">
-        <color rgba="0.8 0.8 0.8 1"/>
+      <material name="light_black">
+        <color rgba="0.15 0.15 0.15 1"/>
       </material>
     </visual>

File: warrior_description/xacro/sensors/imu.xacro (robot description, xacro)
@@ -1,8 +1,12 @@
 <?xml version="1.0"?>
 <robot xmlns:xacro="http://www.ros.org/wiki/xacro" >
+  <!-- ========== IMU Macro ========== -->
+  <xacro:property name="imu_length" value="0.05"/>
+  <xacro:property name="imu_width" value="0.05"/>
+  <xacro:property name="imu_height" value="0.02"/>
   <joint name="imu_joint" type="fixed">
     <parent link="base_link"/>
     <child link ="imu_link"/>
-    <origin xyz="${base_length / 2} 0 ${base_height + imu_height}" rpy="0 0 0"/>
+    <origin xyz="0 0 0" rpy="0 0 0"/>
   </joint>
   <link name="imu_link">
@@ -36,3 +40,14 @@
     </sensor>
   </gazebo>
+  <gazebo>
+    <!-- Odometry Publisher -->
+    <plugin
+      filename="ignition-gazebo-odometry-publisher-system"
+      name="ignition::gazebo::systems::OdometryPublisher">
+      <odom_frame>odom</odom_frame>
+      <robot_base_frame>base_footprint</robot_base_frame>
+      <odom_topic>/odom_gt</odom_topic>
+      <odom_publish_frequency>50</odom_publish_frequency>
+    </plugin>
+  </gazebo>
 </robot>

File: warrior_description/xacro/sensors/lidar.xacro (robot description, xacro)
@@ -48,8 +48,8 @@
             </horizontal>
             <vertical>
-              <samples>30</samples>
+              <samples>40</samples>
               <resolution>1</resolution>
               <min_angle>0</min_angle>
-              <max_angle>0.541799</max_angle>
+              <max_angle>0.501799</max_angle>
             </vertical>
           </scan>

File: warrior_description/xacro/swerve_module/constant.xacro (robot description, xacro)
@@ -1,10 +1,9 @@
 <?xml version="1.0"?>
 <robot xmlns:xacro="http://www.ros.org/wiki/xacro">
-   <!-- <xacro:include filename="$(find warrior_description)/xacro/material.xacro"/> -->
-   <xacro:property name="slewing_plate_mass" value="0.5"/>
+   <xacro:property name="slewing_plate_mass" value="6.0"/>
    <xacro:property name="steer_assembly_mass" value="0.7"/>
-   <xacro:property name="steer_assembly_color" value="light_gray"/>
+   <xacro:property name="steer_assembly_color" value="gray"/>
    <xacro:property name="slewing_plate_color" value="silver"/>
-   <xacro:property name="drive_wheel_color" value="cyan"/>
+   <xacro:property name="drive_wheel_color" value="black"/>
    <xacro:property name="swerve_offset_to_plate" value="0 0 -0.011"/>
    <xacro:property name="drive_wheel_offset" value="0.025 0 -0.147"/>

Commit message: Update Warrior URDF model

File: warrior_description/xacro/material.xacro (robot description, xacro)
@@ -9,8 +9,14 @@
   </material>
   <material name="medium_gray">
-    <color rgba="0.55 0.55 0.55 1"/>
+    <color rgba="0.57 0.58 0.59 1"/>
   </material>
   <material name="light_gray">
     <color rgba="0.8 0.8 0.8 1"/>
+  </material>
+  <material name="metal_gray">
+    <color rgba="0.35 0.35 0.38 1"/>
+  </material>
+  <material name="wood">
+    <color rgba="0.65 0.50 0.39 1.0"/>
   </material>
   <material name="white">
@@ -68,4 +74,7 @@
     <color rgba="0.75 0.75 0.75 1"/>
   </material>
+  <material name="space_gray">
+    <color rgba="0.68 0.68 0.7 1"/>
+  </material>
   <material name="gold">
     <color rgba="1.0 0.84 0.0 1"/>

File: warrior_description/xacro/robot.xacro (robot description, xacro)
@@ -9,8 +9,12 @@
   <!-- <xacro:include filename="$(find warrior_description)/xacro/sensors/gps.xacro"/> -->
   <!-- ========== Properties ========== -->
-  <xacro:property name="angle_offset" value="${pi/6}"/>
-   <xacro:property name="front_plate_offset" value="0.838 0.003 -0.349"/>
-   <xacro:property name="left_plate_offset" value="0.025 0.47 -0.349"/>
-   <xacro:property name="right_plate_offset" value="0.024 -0.468 -0.349"/>
+  <xacro:property name="front_rpy_offset" value="0 0 -${pi/2}"/>
+  <xacro:property name="left_rpy_offset" value="0 0 ${pi/6}"/>
+  <xacro:property name="right_rpy_offset" value="0 0 ${-pi/6 - pi}"/>
+  <xacro:property name="front_xyz_offset" value="0.852889 0.002164 -0.3615845"/>
+  <xacro:property name="left_xyz_offset" value="0.035531 0.474066 -0.3615845"/>
+  <xacro:property name="right_xyz_offset" value="0.035468 -0.469762 -0.3615845"/>
+  <xacro:property name="payload_xyz_offset" value="0.433705 -0.098151 -0.155475"/>
+  <xacro:property name="payload_rpy_offset" value="${pi/2} -${pi} -${pi/2}"/>
   <!-- Wheel properties -->
   <!-- <xacro:property name="wheel_mass" value="2.5"/> -->
@@ -21,14 +25,14 @@
   <!-- <xacro:property name="base_mass" value="6.0"/> -->
   <xacro:property name="base_mass" value="10.0"/>
-  <xacro:property name="base_footprint_height" value="${0.508 + wheel_radius}"/>
+  <xacro:property name="base_footprint_height" value="0.640773"/>
   <!-- Initial orientations (radians) -->
   <xacro:property name="front_initial_angle" value="${pi/2}"/>   <!-- forwarding -->
-  <xacro:property name="left_initial_angle" value="${pi/3}"/>    <!-- forwarding -->
-  <xacro:property name="right_initial_angle" value="-${pi/3 + pi}"/>  <!-- forwarding -->
+  <xacro:property name="left_initial_angle" value="-${pi/6}"/>    <!-- forwarding -->
+  <xacro:property name="right_initial_angle" value="${pi/6 + pi}"/>  <!-- forwarding -->
   <!-- lidar properties -->
   <xacro:property name="pole_height" value="0.527"/>
   <xacro:property name="lidar_offset" value="0.135 -0.005 0.075"/>
   <!-- camera properties -->
-  <xacro:property name="camera_offset" value="0.415 0.0 -0.015"/>
+  <xacro:property name="camera_offset" value="0.425 0.0 -0.015"/>
   <!-- ========== Base Footprint Link ========== -->
   <link name="base_footprint"/>
@@ -45,5 +49,6 @@
         <mesh filename="file://$(find warrior_description)/meshes/warrior_body.stl"/>
       </geometry>
-      <material name="medium_gray"/>
+      <!-- <material name="medium_gray"/> -->
+      <material name="space_gray"/>
     </visual>
     <collision>
@@ -58,4 +63,28 @@
     </inertial>
   </link>
+  <!-- =================== Payload =================== -->
+  <joint name="base_to_payload" type="fixed">
+    <parent link="base_link"/>
+    <child link="payload_link"/>
+    <origin xyz="${payload_xyz_offset}" rpy="${payload_rpy_offset}"/>
+  </joint>
+  <link name="payload_link">
+    <visual>
+      <geometry>
+        <mesh filename="file://$(find warrior_description)/meshes/payload.stl"/>
+      </geometry>
+      <material name="wood"/>
+    </visual>
+    <collision>
+      <geometry>
+        <mesh filename="file://$(find warrior_description)/meshes/payload.stl"/>
+      </geometry>
+    </collision>
+    <inertial>
+      <origin xyz="0 0 0" rpy="0 0 0"/>
+      <mass value="2.0"/>
+      <inertia ixx="0.01" ixy="0" ixz="0" iyy="0.01" iyz="0" izz="0.01"/>
+    </inertial>
+  </link>
   <!-- ========== Instantiate Swerve Modules ========== -->
   <!-- Front Plate Joint -->
@@ -63,5 +92,5 @@
     <parent link="base_link"/>
     <child link="front_slewing_plate_link"/>
-    <origin xyz="${front_plate_offset}" rpy="0 0 0"/>
+    <origin xyz="${front_xyz_offset}" rpy="${front_rpy_offset}"/>
   </joint>
   <!-- Front Swerve Module -->
@@ -71,5 +100,5 @@
     <parent link="base_link"/>
     <child link="left_slewing_plate_link"/>
-    <origin xyz="${left_plate_offset}" rpy="0 0 ${angle_offset}"/>
+    <origin xyz="${left_xyz_offset}" rpy="${left_rpy_offset}"/>
   </joint>
   <!-- Left Swerve Module -->
@@ -79,5 +108,5 @@
     <parent link="base_link"/>
     <child link="right_slewing_plate_link"/>
-    <origin xyz="${right_plate_offset}" rpy="0 0 ${-angle_offset}"/>
+    <origin xyz="${right_xyz_offset}" rpy="${right_rpy_offset}"/>
   </joint>
   <!-- Right Swerve Module -->

File: warrior_description/xacro/ros2_control/gzsim.ros2_control.xacro (robot description, xacro)
@@ -45,5 +45,5 @@
     <gazebo>
         <plugin filename="libgz_ros2_control-system.so" name="gz_ros2_control::GazeboSimROS2ControlPlugin">
-            <parameters>$(find warrior_control)/config/warrior_controllers.yaml</parameters>
+            <parameters>$(find warrior_control)/config/warrior_controllers_sim.yaml</parameters>
         </plugin>
         <plugin filename="gz-sim-imu-system" name="gz::sim::systems::Imu"/>

File: warrior_description/xacro/swerve_module/constant.xacro (robot description, xacro)
@@ -1,13 +1,13 @@
 <?xml version="1.0"?>
 <robot xmlns:xacro="http://www.ros.org/wiki/xacro">
-   <xacro:property name="slewing_plate_mass" value="6.0"/>
-   <xacro:property name="steer_assembly_mass" value="0.7"/>
-   <xacro:property name="steer_assembly_color" value="gray"/>
-   <xacro:property name="slewing_plate_color" value="silver"/>
-   <xacro:property name="drive_wheel_color" value="black"/>
-   <xacro:property name="swerve_offset_to_plate" value="0 0 -0.011"/>
-   <xacro:property name="drive_wheel_offset" value="0.025 0 -0.147"/>
+    <xacro:property name="slewing_plate_mass" value="20.0"/>
+    <xacro:property name="steer_assembly_mass" value="0.7"/>
+    <xacro:property name="steer_assembly_color" value="metal_gray"/>
+    <xacro:property name="slewing_plate_color" value="medium_gray"/>
+    <xacro:property name="drive_wheel_color" value="black"/>
+    <xacro:property name="steer_offset_to_plate" value="0.03175 0 0.077866"/>
+    <xacro:property name="drive_offset_to_steer" value="0.000847 -0.006293 -0.248866"/>
     <xacro:property name="drive_rpy" value="0 0 0"/>
-    <xacro:property name="drive_axis" value="1 0 0"/>
+    <xacro:property name="drive_axis" value="0 1 0"/>
     <!-- ========== Inertia Macros ========== -->
     <xacro:macro name="wheel_inertia" params="mass">

File: warrior_description/xacro/swerve_module/swerve_module.xacro (robot description, xacro)
@@ -7,5 +7,5 @@
     <link name="${prefix}_slewing_plate_link">
       <visual>
-        <origin xyz="0 0 0" rpy="${pi} 0 ${pi}"/>
+        <origin xyz="0 0 0" rpy="0 0 0"/>
         <geometry>
           <mesh filename="file://$(find warrior_description)/meshes/slewing_plate.stl"/>
@@ -14,5 +14,5 @@
       </visual>
       <collision>
-        <origin xyz="0 0 0" rpy="${pi} 0 ${pi}"/>
+        <origin xyz="0 0 0" rpy="0 0 0"/>
         <geometry>
           <mesh filename="file://$(find warrior_description)/meshes/slewing_plate.stl"/>
@@ -25,5 +25,5 @@
       <parent link="${prefix}_slewing_plate_link"/>
       <child link="${prefix}_steer_assembly_link"/>
-      <origin xyz="${swerve_offset_to_plate}" rpy="0 0 ${initial_yaw}"/>
+      <origin xyz="${steer_offset_to_plate}" rpy="0 0 ${initial_yaw}"/>
       <axis xyz="0 0 1"/>
     </joint>
@@ -47,5 +47,5 @@
       <parent link="${prefix}_steer_assembly_link"/>
       <child link="${prefix}_drive_wheel_link"/>
-      <origin xyz="${drive_wheel_offset}" rpy="${drive_rpy}"/>
+      <origin xyz="${drive_offset_to_steer}" rpy="${drive_rpy}"/>
       <axis xyz="${drive_axis}"/>
     </joint>
