Commit message: Update the urdf model for diff_drive_controller

File: warrior_description/xacro/robot.xacro (robot description, xacro)
@@ -1,4 +1,4 @@
 <?xml version="1.0"?>
-<robot xmlns:xacro="http://www.ros.org/wiki/xacro">
+<robot name="warrior_robot" xmlns:xacro="http://www.ros.org/wiki/xacro">
   <!-- ========== Properties ========== -->
   <!-- Base properties -->
@@ -59,5 +59,5 @@
   </xacro:macro>
   <!-- ========== Swerve Module Macro ========== -->
-  <xacro:macro name="swerve_module" params="prefix offset_x offset_y initial_yaw steer_color drive_color">
+  <xacro:macro name="swerve_module" params="prefix offset_x offset_y initial_yaw steer_color drive_color drive_rpy drive_axis">
     <!-- Steer Link -->
     <link name="${prefix}_steer_wheel_link">
@@ -101,6 +101,6 @@
       <parent link="${prefix}_steer_wheel_link"/>
       <child link="${prefix}_drive_wheel_link"/>
-      <origin xyz="0 0 ${wheel_offset_z}" rpy="0 0 0"/>
-      <axis xyz="1 0 0"/>
+      <origin xyz="0 0 ${wheel_offset_z}" rpy="${drive_rpy}"/>
+      <axis xyz="${drive_axis}"/>
     </joint>
   </xacro:macro>
@@ -134,11 +134,11 @@
   <!-- ========== Instantiate Swerve Modules ========== -->
   <!-- Left Module -->
-  <xacro:swerve_module prefix="left" offset_x="${left_x}" offset_y="${left_y}"
+  <xacro:swerve_module prefix="left" offset_x="${left_x}" offset_y="${left_y}" drive_rpy="0 0 ${pi}" drive_axis="1 0 0"
     initial_yaw="${left_initial_angle}" steer_color="blue" drive_color="gray"/>
   <!-- Right Module -->
-  <xacro:swerve_module prefix="right" offset_x="${right_x}" offset_y="${right_y}"
+  <xacro:swerve_module prefix="right" offset_x="${right_x}" offset_y="${right_y}" drive_rpy="0 0 ${pi}" drive_axis="1 0 0"
     initial_yaw="${right_initial_angle}" steer_color="green" drive_color="gray"/>
   <!-- Front Module -->
-  <xacro:swerve_module prefix="front" offset_x="${front_x}" offset_y="0"
+  <xacro:swerve_module prefix="front" offset_x="${front_x}" offset_y="0" drive_rpy="0 0 ${pi}" drive_axis="1 0 0"
     initial_yaw="${front_initial_angle}" steer_color="cyan" drive_color="gray"/>
   <!-- ========== Pole Link ========== -->

Commit message: Update xacro

File: warrior_description/xacro/robot.xacro (robot description, xacro)
@@ -1,5 +1,9 @@
 <?xml version="1.0"?>
 <robot name="warrior_robot" xmlns:xacro="http://www.ros.org/wiki/xacro">
+  <xacro:include filename="$(find warrior_description)/xacro/swerve_module/swerve_module.xacro"/>
   <!-- ========== Properties ========== -->
+   <xacro:property name="front_plate_offset" value="0.838 0.003 -0.349"/>
+   <xacro:property name="left_plate_offset" value="0.025 0.47 -0.349"/>
+   <xacro:property name="right_plate_offset" value="0.024 -0.468 -0.349"/>
   <!-- Base properties -->
   <xacro:property name="base_mass" value="5.0"/>
@@ -49,60 +53,4 @@
     <color rgba="1.0 0.0 1.0 1"/>
   </material>
-  <!-- ========== Inertia Macros ========== -->
-  <xacro:macro name="wheel_inertia" params="mass">
-    <inertial>
-      <origin xyz="0 0 0" rpy="0 0 0"/>
-      <mass value="${mass}"/>
-      <inertia ixx="0.01" ixy="0" ixz="0"
-               iyy="0.01" iyz="0" izz="0.01"/>
-    </inertial>
-  </xacro:macro>
-  <!-- ========== Swerve Module Macro ========== -->
-  <xacro:macro name="swerve_module" params="prefix offset_x offset_y initial_yaw steer_color drive_color drive_rpy drive_axis">
-    <!-- Steer Link -->
-    <link name="${prefix}_steer_wheel_link">
-      <visual>
-        <geometry>
-          <mesh filename="file://$(find warrior_description)/meshes/steer_wheel.stl"/>
-        </geometry>
-        <material name="${steer_color}"/>
-      </visual>
-      <collision>
-        <geometry>
-          <mesh filename="file://$(find warrior_description)/meshes/steer_wheel.stl"/>
-        </geometry>
-      </collision>
-      <xacro:wheel_inertia mass="${wheel_mass}"/>
-    </link>
-    <!-- Steer Joint -->
-    <joint name="${prefix}_steer_joint" type="continuous">
-      <parent link="base_link"/>
-      <child link="${prefix}_steer_wheel_link"/>
-      <origin xyz="${offset_x} ${offset_y} 0" rpy="0 0 ${initial_yaw}"/>
-      <axis xyz="0 0 1"/>
-    </joint>
-    <!-- Drive Wheel Link -->
-    <link name="${prefix}_drive_wheel_link">
-      <visual>
-        <geometry>
-          <mesh filename="file://$(find warrior_description)/meshes/drive_wheel.stl"/>
-        </geometry>
-        <material name="${drive_color}"/>
-      </visual>
-      <collision>
-        <geometry>
-          <mesh filename="file://$(find warrior_description)/meshes/drive_wheel.stl"/>
-        </geometry>
-      </collision>
-      <xacro:wheel_inertia mass="${wheel_mass}"/>
-    </link>
-    <!-- Drive Joint -->
-    <joint name="${prefix}_drive_joint" type="continuous">
-      <parent link="${prefix}_steer_wheel_link"/>
-      <child link="${prefix}_drive_wheel_link"/>
-      <origin xyz="0 0 ${wheel_offset_z}" rpy="${drive_rpy}"/>
-      <axis xyz="${drive_axis}"/>
-    </joint>
-  </xacro:macro>
   <!-- ========== Base Footprint Link ========== -->
   <link name="base_footprint"/>
@@ -117,5 +65,5 @@
     <visual>
       <geometry>
-        <mesh filename="file://$(find warrior_description)/meshes/warrior_base_with_pedal.stl"/>
+        <mesh filename="file://$(find warrior_description)/meshes/warrior_body.stl"/>
       </geometry>
       <material name="gray"/>
@@ -123,5 +71,5 @@
     <collision>
       <geometry>
-        <mesh filename="file://$(find warrior_description)/meshes/warrior_base_with_pedal.stl"/>
+        <mesh filename="file://$(find warrior_description)/meshes/warrior_body.stl"/>
       </geometry>
     </collision>
@@ -133,13 +81,31 @@
   </link>
   <!-- ========== Instantiate Swerve Modules ========== -->
-  <!-- Left Module -->
-  <xacro:swerve_module prefix="left" offset_x="${left_x}" offset_y="${left_y}" drive_rpy="0 0 ${pi}" drive_axis="1 0 0"
-    initial_yaw="${left_initial_angle}" steer_color="blue" drive_color="gray"/>
-  <!-- Right Module -->
-  <xacro:swerve_module prefix="right" offset_x="${right_x}" offset_y="${right_y}" drive_rpy="0 0 ${pi}" drive_axis="1 0 0"
-    initial_yaw="${right_initial_angle}" steer_color="green" drive_color="gray"/>
-  <!-- Front Module -->
-  <xacro:swerve_module prefix="front" offset_x="${front_x}" offset_y="0" drive_rpy="0 0 ${pi}" drive_axis="1 0 0"
-    initial_yaw="${front_initial_angle}" steer_color="cyan" drive_color="gray"/>
+  <!-- Front Plate Joint -->
+  <joint name="base_to_front_plate" type="fixed">
+    <parent link="base_link"/>
+    <child link="front_slewing_plate_link"/>
+    <origin xyz="${front_plate_offset}" rpy="0 0 0"/>
+  </joint>
+  <!-- Front Swerve Module -->
+  <xacro:swerve_module prefix="front" initial_yaw="${front_initial_angle}" drive_rpy="0 0 ${pi}"
+    steer_color="cyan" drive_color="gray"/>
+  <!-- Left Plate Joint -->
+  <joint name="base_to_left_plate" type="fixed">
+    <parent link="base_link"/>
+    <child link="left_slewing_plate_link"/>
+    <origin xyz="${left_plate_offset}" rpy="0 0 0"/>
+  </joint>
+  <!-- Left Swerve Module -->
+  <xacro:swerve_module prefix="left" initial_yaw="${left_initial_angle}" drive_rpy="0 0 ${pi}"
+     steer_color="blue" drive_color="gray"/>
+  <!-- Right Plate Joint -->
+  <joint name="base_to_right_plate" type="fixed">
+    <parent link="base_link"/>
+    <child link="right_slewing_plate_link"/>
+    <origin xyz="${right_plate_offset}" rpy="0 0 0"/>
+  </joint>
+  <!-- Right Swerve Module -->
+  <xacro:swerve_module prefix="right" initial_yaw="${right_initial_angle}" drive_rpy="0 0 ${pi}"
+    steer_color="green" drive_color="gray"/>
   <!-- ========== Pole Link ========== -->
   <link name="pole_link">

Commit message: Update xacro

File: warrior_description/xacro/robot.xacro (robot description, xacro)
@@ -1,4 +1,5 @@
 <?xml version="1.0"?>
 <robot name="warrior_robot" xmlns:xacro="http://www.ros.org/wiki/xacro">
+  <xacro:include filename="$(find warrior_description)/xacro/material.xacro"/>
   <xacro:include filename="$(find warrior_description)/xacro/swerve_module/swerve_module.xacro"/>
   <!-- ========== Properties ========== -->
@@ -31,26 +32,4 @@
   <xacro:property name="pole_height" value="0.9"/>
   <xacro:property name="lidar_offset_x" value="0.36"/>
-  <!-- ========== Material Definitions ========== -->
-  <material name="gray">
-    <color rgba="0.5 0.5 0.5 1"/>
-  </material>
-  <material name="blue">
-    <color rgba="0.0 0.0 1.0 1"/>
-  </material>
-  <material name="yellow">
-    <color rgba="1.0 1.0 0.0 1"/>
-  </material>
-  <material name="green">
-    <color rgba="0.0 1.0 0.0 1"/>
-  </material>
-  <material name="red">
-    <color rgba="1.0 0.0 0.0 1"/>
-  </material>
-  <material name="cyan">
-    <color rgba="0.0 1.0 1.0 1"/>
-  </material>
-  <material name="magenta">
-    <color rgba="1.0 0.0 1.0 1"/>
-  </material>
   <!-- ========== Base Footprint Link ========== -->
   <link name="base_footprint"/>

File: warrior_description/xacro/swerve_module/constant.xacro (robot description, xacro)
@@ -2,4 +2,7 @@
 <robot xmlns:xacro="http://www.ros.org/wiki/xacro">
    <xacro:property name="slewing_plate_mass" value="0.5"/>
+   <xacro:property name="steer_assembly_mass" value="0.7"/>
+   <xacro:property name="steer_assembly_color" value="gray"/>
+   <xacro:property name="slewing_plate_color" value="gray"/>
    <xacro:property name="swerve_offset_to_plate" value="0 0 0.011"/>
    <xacro:property name="drive_wheel_offset" value="-0.025 0 0.147"/>

Commit message: Update xacro

File: warrior_description/xacro/robot.xacro (robot description, xacro)
@@ -7,11 +7,11 @@
    <xacro:property name="left_plate_offset" value="0.025 0.47 -0.349"/>
    <xacro:property name="right_plate_offset" value="0.024 -0.468 -0.349"/>
-  <!-- Base properties -->
-  <xacro:property name="base_mass" value="5.0"/>
-  <xacro:property name="base_footprint_height" value="0.25"/>
   <!-- Wheel properties -->
   <xacro:property name="wheel_mass" value="0.5"/>
   <xacro:property name="wheel_offset_z" value="-0.15"/>
   <xacro:property name="wheel_radius" value="0.1"/>
+  <!-- Base properties -->
+  <xacro:property name="base_mass" value="5.0"/>
+  <xacro:property name="base_footprint_height" value="${0.508 + wheel_radius}"/>
   <!-- Module positions -->
   <xacro:property name="left_y" value="0.465"/>
@@ -26,7 +26,7 @@
   <!-- <xacro:property name="right_initial_angle" value="-2.0944"/> -->  <!-- -120° -->
   <!-- <xacro:property name="front_initial_angle" value="-1.5708"/> -->  <!-- -90° -->
-  <xacro:property name="left_initial_angle" value="-1.5708"/>   <!-- -90° -->
-  <xacro:property name="right_initial_angle" value="-1.5708"/>  <!-- -90° -->
-  <xacro:property name="front_initial_angle" value="-1.5708"/>  <!-- -90° -->
+  <xacro:property name="left_initial_angle" value="0"/>   <!-- -90° -->
+  <xacro:property name="right_initial_angle" value="0"/>  <!-- -90° -->
+  <xacro:property name="front_initial_angle" value="0"/>  <!-- -90° -->
   <!-- Sensor properties -->
   <xacro:property name="pole_height" value="0.9"/>
@@ -34,10 +34,10 @@
   <!-- ========== Base Footprint Link ========== -->
   <link name="base_footprint"/>
-    <joint name="base_footprint_joint" type="fixed">
-        <parent link="base_footprint"/>
-        <child link="base_link"/>
-        <origin xyz="0 0 ${base_footprint_height}" rpy="0 0 0"/>
-        <!-- z = wheel_offset_z (0.15) + wheel_radius (0.1) = 0.25 -->
-    </joint>
+  <joint name="base_footprint_joint" type="fixed">
+      <parent link="base_footprint"/>
+      <child link="base_link"/>
+      <origin xyz="0 0 ${base_footprint_height}" rpy="0 0 0"/>
+      <!-- z = wheel_offset_z (0.15) + wheel_radius (0.1) = 0.25 -->
+  </joint>
   <!-- ========== Base Link ========== -->
   <link name="base_link">
@@ -67,5 +67,5 @@
   </joint>
   <!-- Front Swerve Module -->
-  <xacro:swerve_module prefix="front" initial_yaw="${front_initial_angle}" drive_rpy="0 0 ${pi}"
+  <xacro:swerve_module prefix="front" initial_yaw="${front_initial_angle}"
     steer_color="cyan" drive_color="gray"/>
   <!-- Left Plate Joint -->
@@ -76,5 +76,5 @@
   </joint>
   <!-- Left Swerve Module -->
-  <xacro:swerve_module prefix="left" initial_yaw="${left_initial_angle}" drive_rpy="0 0 ${pi}"
+  <xacro:swerve_module prefix="left" initial_yaw="${left_initial_angle}"
      steer_color="blue" drive_color="gray"/>
   <!-- Right Plate Joint -->
@@ -85,5 +85,5 @@
   </joint>
   <!-- Right Swerve Module -->
-  <xacro:swerve_module prefix="right" initial_yaw="${right_initial_angle}" drive_rpy="0 0 ${pi}"
+  <xacro:swerve_module prefix="right" initial_yaw="${right_initial_angle}"
     steer_color="green" drive_color="gray"/>
   <!-- ========== Pole Link ========== -->

File: warrior_description/xacro/swerve_module/constant.xacro (robot description, xacro)
@@ -5,6 +5,7 @@
    <xacro:property name="steer_assembly_color" value="gray"/>
    <xacro:property name="slewing_plate_color" value="gray"/>
-   <xacro:property name="swerve_offset_to_plate" value="0 0 0.011"/>
-   <xacro:property name="drive_wheel_offset" value="-0.025 0 0.147"/>
+   <xacro:property name="swerve_offset_to_plate" value="0 0 -0.011"/>
+   <xacro:property name="drive_wheel_offset" value="0.025 0 -0.147"/>
+    <xacro:property name="drive_rpy" value="0 0 0"/>
     <xacro:property name="drive_axis" value="1 0 0"/>
     <!-- ========== Inertia Macros ========== -->

File: warrior_description/xacro/swerve_module/swerve_module.xacro (robot description, xacro)
@@ -3,8 +3,9 @@
   <xacro:include filename="$(find warrior_description)/xacro/swerve_module/constant.xacro"/>
   <!-- ========== Swerve Module Macro ========== -->
-  <xacro:macro name="swerve_module" params="prefix initial_yaw steer_color drive_color drive_rpy">
+  <xacro:macro name="swerve_module" params="prefix initial_yaw steer_color drive_color">
     <!-- Slewing Plate Link -->
     <link name="${prefix}_slewing_plate_link">
       <visual>
+        <origin xyz="0 0 0" rpy="${pi} 0 ${pi}"/>
         <geometry>
           <mesh filename="file://$(find warrior_description)/meshes/slewing_plate.stl"/>
@@ -13,4 +14,5 @@
       </visual>
       <collision>
+        <origin xyz="0 0 0" rpy="${pi} 0 ${pi}"/>
         <geometry>
           <mesh filename="file://$(find warrior_description)/meshes/slewing_plate.stl"/>
@@ -51,4 +53,5 @@
     <link name="${prefix}_drive_wheel_link">
       <visual>
+       <origin xyz="0 0 0" rpy="0 0 0"/>
         <geometry>
           <mesh filename="file://$(find warrior_description)/meshes/drive_wheel.stl"/>
@@ -57,4 +60,5 @@
       </visual>
       <collision>
+        <origin xyz="0 0 0" rpy="0 0 0"/>
         <geometry>
           <mesh filename="file://$(find warrior_description)/meshes/drive_wheel.stl"/>

Commit message: Update xacro

File: warrior_description/xacro/robot.xacro (robot description, xacro)
@@ -4,4 +4,5 @@
   <xacro:include filename="$(find warrior_description)/xacro/swerve_module/swerve_module.xacro"/>
   <!-- ========== Properties ========== -->
+  <xacro:property name="angle_offset" value="${pi/6}"/>
    <xacro:property name="front_plate_offset" value="0.838 0.003 -0.349"/>
    <xacro:property name="left_plate_offset" value="0.025 0.47 -0.349"/>
@@ -73,5 +74,5 @@
     <parent link="base_link"/>
     <child link="left_slewing_plate_link"/>
-    <origin xyz="${left_plate_offset}" rpy="0 0 0"/>
+    <origin xyz="${left_plate_offset}" rpy="0 0 ${angle_offset}"/>
   </joint>
   <!-- Left Swerve Module -->
@@ -82,5 +83,5 @@
     <parent link="base_link"/>
     <child link="right_slewing_plate_link"/>
-    <origin xyz="${right_plate_offset}" rpy="0 0 0"/>
+    <origin xyz="${right_plate_offset}" rpy="0 0 ${-angle_offset}"/>
   </joint>
   <!-- Right Swerve Module -->

Commit message: Update xacro

File: warrior_description/xacro/robot.xacro (robot description, xacro)
@@ -24,12 +24,9 @@
   <xacro:property name="camera_offset_z" value="-0.09"/>
   <!-- Initial orientations (radians) -->
-  <!-- <xacro:property name="left_initial_angle" value="-1.0472"/> -->   <!-- -60° -->
-  <!-- <xacro:property name="right_initial_angle" value="-2.0944"/> -->  <!-- -120° -->
-  <!-- <xacro:property name="front_initial_angle" value="-1.5708"/> -->  <!-- -90° -->
-  <xacro:property name="left_initial_angle" value="0"/>   <!-- -90° -->
-  <xacro:property name="right_initial_angle" value="0"/>  <!-- -90° -->
-  <xacro:property name="front_initial_angle" value="0"/>  <!-- -90° -->
+  <xacro:property name="left_initial_angle" value="${pi/2}"/>   <!-- 90° -->
+  <xacro:property name="right_initial_angle" value="-${pi/2}"/>  <!-- 90° -->
+  <xacro:property name="front_initial_angle" value="${pi/2}"/>  <!-- 90° -->
   <!-- Sensor properties -->
-  <xacro:property name="pole_height" value="0.9"/>
+  <xacro:property name="pole_height" value="0.535"/>
   <xacro:property name="lidar_offset_x" value="0.36"/>
   <!-- ========== Base Footprint Link ========== -->
@@ -68,6 +65,5 @@
   </joint>
   <!-- Front Swerve Module -->
-  <xacro:swerve_module prefix="front" initial_yaw="${front_initial_angle}"
-    steer_color="cyan" drive_color="gray"/>
+  <xacro:swerve_module prefix="front" initial_yaw="${front_initial_angle}" />
   <!-- Left Plate Joint -->
   <joint name="base_to_left_plate" type="fixed">
@@ -77,6 +73,5 @@
   </joint>
   <!-- Left Swerve Module -->
-  <xacro:swerve_module prefix="left" initial_yaw="${left_initial_angle}"
-     steer_color="blue" drive_color="gray"/>
+  <xacro:swerve_module prefix="left" initial_yaw="${left_initial_angle}" />
   <!-- Right Plate Joint -->
   <joint name="base_to_right_plate" type="fixed">
@@ -86,14 +81,12 @@
   </joint>
   <!-- Right Swerve Module -->
-  <xacro:swerve_module prefix="right" initial_yaw="${right_initial_angle}"
-    steer_color="green" drive_color="gray"/>
-  <!-- ========== Pole Link ========== -->
+  <xacro:swerve_module prefix="right" initial_yaw="${right_initial_angle}" />
+  <!-- =================== Pole Link ==================== -->
   <link name="pole_link">
-    <!-- Visual/collision commented out in original -->
   </link>
   <joint name="base_to_pole" type="fixed">
     <parent link="base_link"/>
     <child link="pole_link"/>
-    <origin xyz="0 0 ${pole_height}" rpy="3.1415 0 0"/>
+    <origin xyz="0 0 ${pole_height}" rpy="${pi} 0 0"/>
   </joint>
   <!-- ========== LiDAR Link ========== -->
@@ -121,7 +114,7 @@
   </link>
   <joint name="lidar_joint" type="fixed">
-    <parent link="base_link"/>
+    <parent link="pole_link"/>
     <child link="lidar_link"/>
-    <origin xyz="0.32 0 0.875" rpy="3.1415 0 0"/>
+    <origin xyz="0.32 0 0.05" rpy="0 0 0"/>
   </joint>
   <!-- ========== Camera Link ========= -->
@@ -149,7 +142,7 @@
   </link>
   <joint name="camera_joint" type="fixed">
-    <parent link="base_link"/>
+    <parent link="pole_link"/>
     <child link="camera_link"/>
-    <origin xyz="0.32 0 ${0.828 + camera_offset_z}" rpy="3.1415 0 0"/>
+    <origin xyz="0.32 0 0" rpy="0 0 0"/>
   </joint>
   <!-- ========== Gazebo LiDAR Sensor ========== -->

File: warrior_description/xacro/swerve_module/constant.xacro (robot description, xacro)
@@ -1,4 +1,5 @@
 <?xml version="1.0"?>
 <robot xmlns:xacro="http://www.ros.org/wiki/xacro">
+  <!-- <xacro:include filename="$(find warrior_description)/xacro/material.xacro"/> -->
    <xacro:property name="slewing_plate_mass" value="0.5"/>
    <xacro:property name="steer_assembly_mass" value="0.7"/>
@@ -7,4 +8,6 @@
    <xacro:property name="swerve_offset_to_plate" value="0 0 -0.011"/>
    <xacro:property name="drive_wheel_offset" value="0.025 0 -0.147"/>
+    <xacro:property name="steer_color" value="cyan"/>
+    <xacro:property name="drive_color" value="gray"/>
     <xacro:property name="drive_rpy" value="0 0 0"/>
     <xacro:property name="drive_axis" value="1 0 0"/>

File: warrior_description/xacro/swerve_module/swerve_module.xacro (robot description, xacro)
@@ -3,5 +3,5 @@
   <xacro:include filename="$(find warrior_description)/xacro/swerve_module/constant.xacro"/>
   <!-- ========== Swerve Module Macro ========== -->
-  <xacro:macro name="swerve_module" params="prefix initial_yaw steer_color drive_color">
+  <xacro:macro name="swerve_module" params="prefix initial_yaw">
     <!-- Slewing Plate Link -->
     <link name="${prefix}_slewing_plate_link">
