Commit message: Add camera support

File: warrior_description/xacro/robot.xacro (robot description, xacro)
@@ -5,4 +5,5 @@
   <xacro:include filename="$(find warrior_description)/xacro/swerve_module/swerve_module.xacro"/>
   <xacro:include filename="$(find warrior_description)/xacro/sensors/lidar.xacro"/>
+  <xacro:include filename="$(find warrior_description)/xacro/sensors/camera.xacro"/>
   <!-- ========== Properties ========== -->
   <xacro:property name="angle_offset" value="${pi/6}"/>
@@ -23,13 +24,16 @@
   <xacro:property name="right_x" value="0.03" />
   <xacro:property name="front_x" value="0.845"/>
-  <!-- Camera -->
-  <xacro:property name="camera_offset_z" value="-0.09"/>
   <!-- Initial orientations (radians) -->
   <xacro:property name="left_initial_angle" value="${pi/2}"/>   <!-- 90° -->
   <xacro:property name="right_initial_angle" value="-${pi/2}"/>  <!-- 90° -->
   <xacro:property name="front_initial_angle" value="${pi/2}"/>  <!-- 90° -->
-  <!-- Sensor properties -->
-  <xacro:property name="pole_height" value="0.535"/>
-  <xacro:property name="lidar_offset_x" value="0.36"/>
+  <!-- lidar properties -->
+  <xacro:property name="pole_height" value="0.527"/>
+  <xacro:property name="lidar_offset_x" value="0.32"/>
+  <xacro:property name="lidar_offset_z" value="0.005"/>
+  <!-- camera properties -->
+  <xacro:property name="camera_offset_x" value="0.32"/>
+  <xacro:property name="camera_offset_y" value="0.0"/>
+  <xacro:property name="camera_offset_z" value="-0.115"/>
   <!-- ========== Base Footprint Link ========== -->
   <link name="base_footprint"/>
@@ -94,32 +98,7 @@
   <!-- ========== LiDAR Sensor ========== -->
   <xacro:lidar_macro parent="pole_link" lidar_name="L1_lidar"
-                     xyz="${lidar_offset_x} 0 0" rpy="0 0 0" mass="0.5"/>
-  <!-- ========== Camera Link ========= -->
-  <link name="camera_link">
-    <visual>
-      <origin xyz="0 -0.027 ${camera_offset_z}" rpy="0 0 0"/>
-      <geometry>
-        <mesh filename="file://$(find warrior_description)/meshes/insta360_camera.stl"/>
-      </geometry>
-      <material name="light_grey">
-        <color rgba="0.8 0.8 0.8 1"/>
-      </material>
-    </visual>
-    <collision>
-      <origin xyz="0 -0.027 ${camera_offset_z}" rpy="0 0 0"/>
-      <geometry>
-        <mesh filename="file://$(find warrior_description)/meshes/insta360_camera.stl"/>
-      </geometry>
-    </collision>
-    <inertial>
-        <origin xyz="0 -0.027 ${camera_offset_z}" rpy="0 0 0"/>
-        <mass value="0.5"/>
-        <inertia ixx="0.005" ixy="0" ixz="0" iyy="0.005" iyz="0" izz="0.002"/>
-    </inertial>
-  </link>
-  <joint name="camera_joint" type="fixed">
-    <parent link="pole_link"/>
-    <child link="camera_link"/>
-    <origin xyz="0.32 0 0" rpy="0 0 0"/>
-  </joint>
+                     xyz="${lidar_offset_x} 0 ${lidar_offset_z}" rpy="0 0 0" mass="0.5"/>
+  <!-- ========== Camera Sensor ========== -->
+  <xacro:camera_macro parent="pole_link" camera_name="insta360_camera"
+                      xyz="${camera_offset_x} ${camera_offset_y} ${camera_offset_z}" rpy="-${pi/2} 0 -${pi/2}" mass="0.5"/>
 </robot>

File: warrior_description/xacro/sensors/camera.xacro (robot description, xacro)
@@ -1,44 +1,52 @@
 <?xml version="1.0"?>
 <robot xmlns:xacro="http://www.ros.org/wiki/xacro" >
-  <joint name="camera_joint" type="fixed">
-    <parent link="chassis"/>
-    <child link ="camera_link"/>
-    <origin xyz="${base_length} 0 ${base_height/2}"/>
-  </joint>
+  <!-- ========== camera Macro ========== -->
+  <xacro:macro name="camera_macro" params="parent camera_name xyz rpy:='0 0 0' mass:=1.0">
   <link name="camera_link">
     <visual>
       <geometry>
-          <box size = "${camera_width} ${camera_length} ${camera_height}"/>
+        <mesh filename="file://$(find warrior_description)/meshes/insta360_camera.stl"/>
       </geometry>
-      <material name="green"/>
+      <material name="light_grey">
+        <color rgba="0.8 0.8 0.8 1"/>
+      </material>
     </visual>
+    <collision>
+      <geometry>
+        <mesh filename="file://$(find warrior_description)/meshes/insta360_camera.stl"/>
+      </geometry>
+    </collision>
+    <inertial>
+        <mass value="${mass}"/>
+        <inertia ixx="0.005" ixy="0" ixz="0" iyy="0.005" iyz="0" izz="0.002"/>
+    </inertial>
   </link>
-  <joint name="camera_optical_joint" type="fixed">
-    <parent link="camera_link"/>
-    <child link ="camera_link_optical"/>
-    <origin xyz="0 0 0" rpy ="${-pi/2} 0 ${-pi/2}"/>
+  <joint name="camera_joint" type="fixed">
+    <parent link="${parent}"/>
+    <child link="camera_link"/>
+    <origin xyz="${xyz}" rpy="${rpy}"/>
   </joint>
-  <link name="camera_link_optical"></link>
-<gazebo reference="camera_link">
-  <material>Gazebo/Green</material>
-  <sensor name="camera" type="camera">
-    <pose>0 0 0 0 0 0</pose>
-    <update_rate>30</update_rate>
-    <camera>
-    <camera_info_topic>/camera/camera_info</camera_info_topic>
-      <horizontal_fov>1.047</horizontal_fov>
-      <image>
-        <width>640</width>
-        <height>480</height>
-        <format>R8G8B8</format>
-      </image>
-      <clip>
-        <near>0.1</near>
-        <far>100</far>
-      </clip>
-    </camera>
-    <topic>/camera/image_raw</topic>
-    <gz_frame_id>camera_link_optical</gz_frame_id>
-  </sensor>
-</gazebo>
+  <gazebo reference="camera_link">
+    <material>Gazebo/GreyTransparent</material>
+    <sensor name="${camera_name}" type="camera">
+      <pose>0 0 0 0 0 0</pose>
+      <update_rate>30</update_rate>
+      <camera>
+      <camera_info_topic>/camera/camera_info</camera_info_topic>
+        <horizontal_fov>1.047</horizontal_fov>
+        <image>
+          <width>640</width>
+          <height>480</height>
+          <format>R8G8B8</format>
+        </image>
+        <clip>
+          <near>0.1</near>
+          <far>100</far>
+        </clip>
+      </camera>
+      <topic>/camera/image_raw</topic>
+      <gz_frame_id>camera_link</gz_frame_id>
+    </sensor>
+  </gazebo>
+  </xacro:macro>
 </robot>

Commit message: Complete stuff

File: warrior_description/xacro/robot.xacro (robot description, xacro)
@@ -18,14 +18,8 @@
   <xacro:property name="base_mass" value="5.0"/>
   <xacro:property name="base_footprint_height" value="${0.508 + wheel_radius}"/>
-  <!-- Module positions -->
-  <xacro:property name="left_y" value="0.465"/>
-  <xacro:property name="right_y" value="-0.465"/>
-  <xacro:property name="left_x" value="0.03" />
-  <xacro:property name="right_x" value="0.03" />
-  <xacro:property name="front_x" value="0.845"/>
   <!-- Initial orientations (radians) -->
-  <xacro:property name="left_initial_angle" value="${pi/2}"/>   <!-- 90° -->
-  <xacro:property name="right_initial_angle" value="-${pi/2}"/>  <!-- 90° -->
-  <xacro:property name="front_initial_angle" value="${pi/2}"/>  <!-- 90° -->
+  <xacro:property name="left_initial_angle" value="${pi/3}"/>    <!-- 90° -->
+  <xacro:property name="right_initial_angle" value="-${pi/3 + pi}"/>  <!-- 90° -->
+  <xacro:property name="front_initial_angle" value="${pi/2}"/>   <!-- 90° -->
   <!-- lidar properties -->
   <xacro:property name="pole_height" value="0.527"/>
@@ -33,7 +27,5 @@
   <xacro:property name="lidar_offset_z" value="0.005"/>
   <!-- camera properties -->
-  <xacro:property name="camera_offset_x" value="0.32"/>
-  <xacro:property name="camera_offset_y" value="0.0"/>
-  <xacro:property name="camera_offset_z" value="-0.115"/>
+  <xacro:property name="camera_offset" value="0.32 0.0 -0.115"/>
   <!-- ========== Base Footprint Link ========== -->
   <link name="base_footprint"/>
@@ -101,4 +93,4 @@
   <!-- ========== Camera Sensor ========== -->
   <xacro:camera_macro parent="pole_link" camera_name="insta360_camera"
-                      xyz="${camera_offset_x} ${camera_offset_y} ${camera_offset_z}" rpy="-${pi/2} 0 -${pi/2}" mass="0.5"/>
+                      xyz="${camera_offset}" rpy="-${pi/2} 0 -${pi/2}" mass="0.5"/>
 </robot>

Commit message: Update README.md

File: warrior_description/xacro/robot.xacro (robot description, xacro)
@@ -19,7 +19,7 @@
   <xacro:property name="base_footprint_height" value="${0.508 + wheel_radius}"/>
   <!-- Initial orientations (radians) -->
-  <xacro:property name="left_initial_angle" value="${pi/3}"/>    <!-- 90° -->
-  <xacro:property name="right_initial_angle" value="-${pi/3 + pi}"/>  <!-- 90° -->
-  <xacro:property name="front_initial_angle" value="${pi/2}"/>   <!-- 90° -->
+  <xacro:property name="front_initial_angle" value="${pi/2}"/>   <!-- forwarding -->
+  <xacro:property name="left_initial_angle" value="${pi/3}"/>    <!-- forwarding -->
+  <xacro:property name="right_initial_angle" value="-${pi/3 + pi}"/>  <!-- forwarding -->
   <!-- lidar properties -->
   <xacro:property name="pole_height" value="0.527"/>

Commit message: Add camera support in Gazebo

File: warrior_description/xacro/robot.xacro (robot description, xacro)
@@ -93,4 +93,4 @@
   <!-- ========== Camera Sensor ========== -->
   <xacro:camera_macro parent="pole_link" camera_name="insta360_camera"
-                      xyz="${camera_offset}" rpy="-${pi/2} 0 -${pi/2}" mass="0.5"/>
+                      xyz="${camera_offset}" rpy="${pi} 0 0" mass="0.5"/>
 </robot>

File: warrior_description/xacro/sensors/camera.xacro (robot description, xacro)
@@ -5,4 +5,5 @@
   <link name="camera_link">
     <visual>
+      <origin xyz="0 0 0" rpy="${pi/2} 0 -${pi/2}"/>
       <geometry>
         <mesh filename="file://$(find warrior_description)/meshes/insta360_camera.stl"/>
@@ -13,4 +14,5 @@
     </visual>
     <collision>
+      <origin xyz="0 0 0" rpy="${pi/2} 0 -${pi/2}"/>
       <geometry>
         <mesh filename="file://$(find warrior_description)/meshes/insta360_camera.stl"/>

Commit message: Update course map

File: warrior_description/xacro/robot.xacro (robot description, xacro)
@@ -16,5 +16,5 @@
   <xacro:property name="wheel_radius" value="0.1"/>
   <!-- Base properties -->
-  <xacro:property name="base_mass" value="5.0"/>
+  <xacro:property name="base_mass" value="0.5"/>
   <xacro:property name="base_footprint_height" value="${0.508 + wheel_radius}"/>
   <!-- Initial orientations (radians) -->

Commit message: Update physics property in xacro

File: warrior_description/xacro/robot.xacro (robot description, xacro)
@@ -17,12 +17,11 @@
   <xacro:property name="payload_xyz_offset" value="0.433705 -0.098151 -0.155475"/>
   <xacro:property name="payload_rpy_offset" value="${pi/2} -${pi} -${pi/2}"/>
+  <xacro:property name="payload_mass" value="9.5"/>
   <!-- Wheel properties -->
-  <!-- <xacro:property name="wheel_mass" value="2.5"/> -->
   <xacro:property name="wheel_mass" value="5.0"/>
-  <xacro:property name="wheel_offset_z" value="-0.15"/>
-  <xacro:property name="wheel_radius" value="0.1"/>
+  <xacro:property name="wheel_radius" value="0.025"/>
   <!-- Base properties -->
   <!-- <xacro:property name="base_mass" value="6.0"/> -->
-  <xacro:property name="base_mass" value="10.0"/>
+  <xacro:property name="base_mass" value="25.0"/>
   <xacro:property name="base_footprint_height" value="0.640773"/>
   <!-- Initial orientations (radians) -->
@@ -41,5 +40,4 @@
       <child link="base_link"/>
       <origin xyz="0 0 ${base_footprint_height}" rpy="0 0 0"/>
-      <!-- z = wheel_offset_z (0.15) + wheel_radius (0.1) = 0.25 -->
   </joint>
   <!-- ========== Base Link ========== -->
@@ -83,5 +81,5 @@
     <inertial>
       <origin xyz="0 0 0" rpy="0 0 0"/>
-      <mass value="2.0"/>
+      <mass value="${payload_mass}"/>
       <inertia ixx="0.01" ixy="0" ixz="0" iyy="0.01" iyz="0" izz="0.01"/>
     </inertial>

File: warrior_description/xacro/swerve_module/constant.xacro (robot description, xacro)
@@ -1,6 +1,6 @@
 <?xml version="1.0"?>
 <robot xmlns:xacro="http://www.ros.org/wiki/xacro">
-    <xacro:property name="slewing_plate_mass" value="20.0"/>
-    <xacro:property name="steer_assembly_mass" value="0.7"/>
+    <xacro:property name="slewing_plate_mass" value="15.0"/>
+    <xacro:property name="steer_assembly_mass" value="6.0"/>
     <xacro:property name="steer_assembly_color" value="metal_gray"/>
     <xacro:property name="slewing_plate_color" value="medium_gray"/>

Commit message: added gps to robot xacro, plugin to competition world

File: warrior_description/xacro/robot.xacro (robot description, xacro)
@@ -7,5 +7,5 @@
   <xacro:include filename="$(find warrior_description)/xacro/sensors/camera.xacro"/>
   <xacro:include filename="$(find warrior_description)/xacro/sensors/imu.xacro"/>
-  <!-- <xacro:include filename="$(find warrior_description)/xacro/sensors/gps.xacro"/> -->
+  <xacro:include filename="$(find warrior_description)/xacro/sensors/gps.xacro"/>
   <!-- ========== Properties ========== -->
   <xacro:property name="front_rpy_offset" value="0 0 -${pi/2}"/>
@@ -124,4 +124,6 @@
   <xacro:camera_macro parent="pole_link" camera_name="insta360_camera"
                       xyz="${camera_offset}" rpy="${pi} 0 0" mass="0.5"/>
+  <!-- ========== GPS =========== -->
+  <xacro:gps_macro parent="pole_link" xyz="0 0 0"/>
   <!-- ========== Beacon Light ========== -->
   <link name="beacon_light_link">

File: warrior_description/xacro/sensors/gps.xacro (robot description, xacro)
@@ -1,18 +1,20 @@
 <?xml version="1.0"?>
 <robot xmlns:xacro="http://www.ros.org/wiki/xacro" >
-  <joint name="navsat_joint" type="fixed">
-    <origin xyz="0 0 0" rpy="0 0 0" />
-    <parent link="base_link"/>
-    <child link="navsat_link" />
-  </joint>
-  <link name="navsat_link">
-  </link>
-  <gazebo reference="navsat_link">
-    <sensor name="navsat" type="navsat">
-      <always_on>1</always_on>
-      <update_rate>1</update_rate>
-      <topic>navsat</topic>
-      <gz_frame_id>navsat_link</gz_frame_id>
-    </sensor>
-  </gazebo>
+  <xacro:macro name="gps_macro" params = "parent, xyz">
+    <joint name="navsat_joint" type="fixed">
+      <origin xyz="${xyz}" rpy="0 0 0" />
+      <parent link="${parent}"/>
+      <child link="navsat_link" />
+    </joint>
+    <link name="navsat_link">
+    </link>
+    <gazebo reference="navsat_link">
+      <sensor name="navsat" type="navsat">
+        <always_on>1</always_on>
+        <update_rate>1</update_rate>
+        <topic>navsat</topic>
+        <gz_frame_id>navsat_link</gz_frame_id>
+      </sensor>
+    </gazebo>
+  </xacro:macro>
 </robot>

Commit message: integrate real sensor topics into nav

File: warrior_description/xacro/robot.xacro (robot description, xacro)
@@ -125,5 +125,6 @@
                       xyz="${camera_offset}" rpy="${pi} 0 0" mass="0.5"/>
   <!-- ========== GPS =========== -->
-  <xacro:gps_macro parent="pole_link" xyz="0 0 0"/>
+  <xacro:gps_macro parent="pole_link" name="navsat1" xyz="0.27 0 0"/>
+  <xacro:gps_macro parent="base_link" name="navsat2" xyz="0.76 0 0"/>
   <!-- ========== Beacon Light ========== -->
   <link name="beacon_light_link">

File: warrior_description/xacro/sensors/gps.xacro (robot description, xacro)
@@ -1,6 +1,6 @@
 <?xml version="1.0"?>
 <robot xmlns:xacro="http://www.ros.org/wiki/xacro" >
-  <xacro:macro name="gps_macro" params = "parent xyz">
-    <joint name="navsat_joint" type="fixed">
+  <xacro:macro name="gps_macro" params = "parent name xyz">
+    <joint name="${name}_link" type="fixed">
       <origin xyz="${xyz}" rpy="0 0 0" />
       <parent link="${parent}"/>

Commit message: Complete lidar changes

File: warrior_description/xacro/robot.xacro (robot description, xacro)
@@ -120,5 +120,19 @@
   <!-- ========== LiDAR Sensor ========== -->
   <xacro:lidar_macro parent="pole_link" lidar_name="L1_lidar"
-                     xyz="${lidar_offset}" rpy="0 0 3.1415" mass="0.5"/>
+                     xyz="${lidar_offset}" rpy="0 0 0" mass="0.5"/>
+  <joint name="unilidar_imu_joint" type="fixed">
+    <parent link="L1_lidar_link"/>
+    <child link="unilidar_imu"/>
+    <origin xyz="0 0 0" rpy="0 0 0"/>
+  </joint>
+  <joint name="unilidar_lidar_joint" type="fixed">
+    <parent link="unilidar_imu"/>
+    <child link="unilidar_lidar"/>
+    <origin xyz="0 0 0" rpy="0 0 0"/>
+  </joint>
+  <link name="unilidar_imu">
+  </link>
+  <link name="unilidar_lidar">
+  </link>
   <!-- ========== Camera Sensor ========== -->
   <xacro:camera_macro parent="pole_link" camera_name="insta360_camera"

File: warrior_description/xacro/sensors/gps.xacro (robot description, xacro)
@@ -5,14 +5,14 @@
       <origin xyz="${xyz}" rpy="0 0 0" />
       <parent link="${parent}"/>
-      <child link="navsat_link" />
+      <child link="${name}_link" />
     </joint>
-    <link name="navsat_link">
+    <link name="${name}_link">
     </link>
-    <gazebo reference="navsat_link">
+    <gazebo reference="${name}_link">
       <sensor name="navsat" type="navsat">
         <always_on>1</always_on>
         <update_rate>1</update_rate>
         <topic>navsat</topic>
-        <gz_frame_id>navsat_link</gz_frame_id>
+        <gz_frame_id>${name}_link</gz_frame_id>
       </sensor>
     </gazebo>

Commit message: jazzy branch

File: warrior_description/xacro/robot.xacro (robot description, xacro)
@@ -139,6 +139,6 @@
                       xyz="${camera_offset}" rpy="${pi} 0 0" mass="0.5"/>
   <!-- ========== GPS =========== -->
-  <xacro:gps_macro parent="pole_link" name="navsat1" xyz="0.27 0 0"/>
-  <xacro:gps_macro parent="base_link" name="navsat2" xyz="0.76 0 0"/>
+  <xacro:gps_macro parent="pole_link" gps_name="navsat1" xyz="0.27 0 0"/>
+  <xacro:gps_macro parent="base_link" gps_name="navsat2" xyz="0.76 0 0"/>
   <!-- ========== Beacon Light ========== -->
   <link name="beacon_light_link">

File: warrior_description/xacro/sensors/gps.xacro (robot description, xacro)
@@ -1,18 +1,18 @@
 <?xml version="1.0"?>
 <robot xmlns:xacro="http://www.ros.org/wiki/xacro" >
-  <xacro:macro name="gps_macro" params = "parent name xyz">
-    <joint name="${name}_link" type="fixed">
+  <xacro:macro name="gps_macro" params = "parent gps_name xyz">
+    <joint name="${gps_name}_joint" type="fixed">
       <origin xyz="${xyz}" rpy="0 0 0" />
       <parent link="${parent}"/>
-      <child link="${name}_link" />
+      <child link="${gps_name}_link" />
     </joint>
-    <link name="${name}_link">
+    <link name="${gps_name}_link">
     </link>
-    <gazebo reference="${name}_link">
-      <sensor name="navsat" type="navsat">
+    <gazebo reference="${gps_name}_link">
+      <sensor name="${gps_name}" type="navsat">
         <always_on>1</always_on>
         <update_rate>1</update_rate>
-        <topic>navsat</topic>
-        <gz_frame_id>${name}_link</gz_frame_id>
+        <topic>${gps_name}</topic>
+        <gz_frame_id>${gps_name}_link</gz_frame_id>
       </sensor>
     </gazebo>

File: warrior_description/xacro/sensors/lidar.xacro (robot description, xacro)
@@ -44,6 +44,6 @@
               <samples>360</samples>
               <resolution>1</resolution>
-              <min_angle>0.4</min_angle>
-              <max_angle>6.0</max_angle>
+              <min_angle>0.0</min_angle>
+              <max_angle>6.28</max_angle>
             </horizontal>
             <vertical>

Commit message: Remove dependencies

File: warrior_description/xacro/robot.xacro (robot description, xacro)
@@ -139,6 +139,6 @@
                       xyz="${camera_offset}" rpy="${pi} 0 0" mass="0.5"/>
   <!-- ========== GPS =========== -->
-  <xacro:gps_macro parent="pole_link" name="navsat1" xyz="0.27 0 0"/>
-  <xacro:gps_macro parent="base_link" name="navsat2" xyz="0.76 0 0"/>
+  <xacro:gps_macro parent="pole_link" name="gps1" xyz="0.27 0 0"/>
+  <xacro:gps_macro parent="base_link" name="gps2" xyz="0.76 0 0"/>
   <!-- ========== Beacon Light ========== -->
   <link name="beacon_light_link">

File: warrior_description/xacro/sensors/gps.xacro (robot description, xacro)
@@ -2,17 +2,17 @@
 <robot xmlns:xacro="http://www.ros.org/wiki/xacro" >
   <xacro:macro name="gps_macro" params = "parent name xyz">
-    <joint name="${name}_link" type="fixed">
+    <joint name="${name}_joint" type="fixed">
       <origin xyz="${xyz}" rpy="0 0 0" />
       <parent link="${parent}"/>
-      <child link="${name}_link" />
+      <child link="${name}" />
     </joint>
-    <link name="${name}_link">
+    <link name="${name}">
     </link>
-    <gazebo reference="${name}_link">
-      <sensor name="navsat" type="navsat">
+    <gazebo reference="${name}">
+      <sensor name="${name}" type="navsat">
         <always_on>1</always_on>
         <update_rate>1</update_rate>
         <topic>navsat</topic>
-        <gz_frame_id>${name}_link</gz_frame_id>
+        <gz_frame_id>${name}</gz_frame_id>
       </sensor>
     </gazebo>

Commit message: Finetuned the costmap

File: warrior_description/xacro/robot.xacro (robot description, xacro)
@@ -135,10 +135,12 @@
   <link name="unilidar_lidar">
   </link>
+  <!-- <link name="unilidar_imu_initial">
+  </link> -->
   <!-- ========== Camera Sensor ========== -->
   <xacro:camera_macro parent="pole_link" camera_name="insta360_camera"
                       xyz="${camera_offset}" rpy="${pi} 0 0" mass="0.5"/>
   <!-- ========== GPS =========== -->
-  <xacro:gps_macro parent="pole_link" name="gps1" xyz="0.27 0 0"/>
-  <xacro:gps_macro parent="base_link" name="gps2" xyz="0.76 0 0"/>
+  <xacro:gps_macro parent="pole_link" name="gps2" xyz="0.27 0 0"/>
+  <xacro:gps_macro parent="base_link" name="gps1" xyz="0.76 0 0"/>
   <!-- ========== Beacon Light ========== -->
   <link name="beacon_light_link">

Commit message: phone sensors and param updates

File: warrior_description/xacro/robot.xacro (robot description, xacro)
@@ -135,9 +135,14 @@
   <link name="unilidar_lidar">
   </link>
+  <joint name="imu_joint" type="fixed">
+    <parent link="base_link"/>
+    <child link="imu_frame"/>
+    <origin xyz="0.04 0 0" rpy = "0 0 0"/>
+  </joint>
   <!-- ========== Camera Sensor ========== -->
   <xacro:camera_macro parent="pole_link" camera_name="insta360_camera"
                       xyz="${camera_offset}" rpy="${pi} 0 0" mass="0.5"/>
   <!-- ========== GPS =========== -->
-  <xacro:gps_macro parent="pole_link" gps_name="gps2" xyz="0.27 0 0"/>
+  <xacro:gps_macro parent="base_link" gps_name="gps_frame" xyz="0.04 0 0"/>
   <xacro:gps_macro parent="base_link" gps_name="gps1" xyz="0.76 0 0"/>
   <!-- ========== Beacon Light ========== -->
