Commit message: phone sensor and nav2 param updates

File: warrior_description/xacro/robot.xacro (robot description, xacro)
@@ -135,14 +135,9 @@
   <link name="unilidar_lidar">
   </link>
-  <joint name="imu_joint" type="fixed">
-    <parent link="base_link"/>
-    <child link="imu_frame"/>
-    <origin xyz="0.04 0 0" rpy = "0 0 0"/>
-  </joint>
   <!-- ========== Camera Sensor ========== -->
   <xacro:camera_macro parent="pole_link" camera_name="insta360_camera"
                       xyz="${camera_offset}" rpy="${pi} 0 0" mass="0.5"/>
   <!-- ========== GPS =========== -->
-  <xacro:gps_macro parent="base_link" gps_name="gps_frame" xyz="0.04 0 0"/>
+  <xacro:gps_macro parent="base_link" gps_name="gps" xyz="0.04 0 0"/>
   <xacro:gps_macro parent="base_link" gps_name="gps1" xyz="0.76 0 0"/>
   <!-- ========== Beacon Light ========== -->

File: warrior_description/xacro/sensors/gps.xacro (robot description, xacro)
@@ -5,14 +5,14 @@
       <origin xyz="${xyz}" rpy="0 0 0" />
       <parent link="${parent}"/>
-      <child link="${gps_name}_link" />
+      <child link="${gps_name}_frame" />
     </joint>
-    <link name="${gps_name}_link">
+    <link name="${gps_name}_frame">
     </link>
-    <gazebo reference="${gps_name}_link">
+    <gazebo reference="${gps_name}_frame">
       <sensor name="${gps_name}" type="navsat">
         <always_on>1</always_on>
         <update_rate>1</update_rate>
         <topic>${gps_name}</topic>
-        <gz_frame_id>${gps_name}_link</gz_frame_id>
+        <gz_frame_id>${gps_name}_frame</gz_frame_id>
       </sensor>
     </gazebo>

File: warrior_description/xacro/sensors/imu.xacro (robot description, xacro)
@@ -7,8 +7,8 @@
   <joint name="imu_joint" type="fixed">
     <parent link="base_link"/>
-    <child link ="imu_link"/>
+    <child link ="imu_frame"/>
     <origin xyz="0 0 0" rpy="0 0 0"/>
   </joint>
-  <link name="imu_link">
+  <link name="imu_frame">
     <visual>
       <geometry>
@@ -18,5 +18,5 @@
     </visual>
   </link>
-  <gazebo reference="imu_link">
+  <gazebo reference="imu_frame">
     <sensor name="imu_sensor" type="imu">
       <pose>0 0 0 0 0 0</pose>
@@ -37,5 +37,5 @@
       </imu>
       <topic>imu</topic>
-      <gz_frame_id>imu_link</gz_frame_id>
+      <gz_frame_id>imu_frame</gz_frame_id>
     </sensor>
   </gazebo>
