Commit message: adds working nav2 goal

File: warrior_description/xacro/robot.xacro (robot description, xacro)
@@ -24,4 +24,7 @@
   <!-- <xacro:property name="base_mass" value="6.0"/> -->
   <xacro:property name="base_mass" value="25.0"/>
+  <!-- Locate base_footprint at the centroid of the three swerve modules. -->
+  <xacro:property name="base_footprint_x_offset" value="-0.307963"/>
+  <xacro:property name="base_footprint_y_offset" value="-0.002156"/>
   <xacro:property name="base_footprint_height" value="0.640773"/>
   <!-- Initial orientations (radians) -->
@@ -39,5 +42,5 @@
       <parent link="base_footprint"/>
       <child link="base_link"/>
-      <origin xyz="0 0 ${base_footprint_height}" rpy="0 0 0"/>
+      <origin xyz="${base_footprint_x_offset} ${base_footprint_y_offset} ${base_footprint_height}" rpy="0 0 0"/>
   </joint>
   <!-- ========== Base Link ========== -->
