Commit message: killed evil comma

File: warrior_description/xacro/sensors/gps.xacro (robot description, xacro)
@@ -1,5 +1,5 @@
 <?xml version="1.0"?>
 <robot xmlns:xacro="http://www.ros.org/wiki/xacro" >
-  <xacro:macro name="gps_macro" params = "parent, xyz">
+  <xacro:macro name="gps_macro" params = "parent xyz">
     <joint name="navsat_joint" type="fixed">
       <origin xyz="${xyz}" rpy="0 0 0" />
